File: lh60.sch (KiCad schematic (older format))
At the start: 7 parts

Commit message: 20220311
Changed lines of the file:
@@
 	1600 4500 1700 4500
 $Sheet
-S 5250 2300 1100 2800
+S 4500 2550 650  2350
 U 622A1CB9
 F0 "Matrix" 50
 F1 "matrix.sch" 50
+F2 "ROW1" I L 4500 2800 50
+F3 "ROW2" I L 4500 2900 50
+F4 "ROW3" I L 4500 3000 50
+F5 "ROW4" I L 4500 3100 50
+F6 "ROW5" I L 4500 3200 50
+F7 "COL1" I L 4500 3350 50
+F8 "COL2" I L 4500 3450 50
+F9 "COL3" I L 4500 3550 50
+F10 "COL4" I L 4500 3650 50
+F11 "COL5" I L 4500 3750 50
+F12 "COL6" I L 4500 3850 50
+F13 "COL7" I L 4500 3950 50
+F14 "COL8" I L 4500 4050 50
+F15 "COL9" I L 4500 4150 50
+F16 "COL10" I L 4500 4250 50
+F17 "COL11" I L 4500 4350 50
+F18 "COL12" I L 4500 4450 50
+F19 "COL13" I L 4500 4550 50
+F20 "COL14" I L 4500 4650 50
 $EndSheet
 $EndSCHEMATC

Commit message: 20220313
Connections:
- net ROW4: now reaches U?.1 (PD3)
- net ROW5: now reaches U?.2 (PD4)
- net ROW1: now reaches U?.30 (PD0)
- net ROW2: now reaches U?.31 (PD1)
- net ROW3: now reaches U?.32 (PD2)
Changed lines of the file:
@@
 F20 "COL14" I L 4500 4650 50
 $EndSheet
+Wire Bus Line
+	4000 4900 4200 4900
+Entry Wire Line
+	3900 4500 4000 4600
+Entry Wire Line
+	3900 4600 4000 4700
+Entry Wire Line
+	3900 4700 4000 4800
+Wire Wire Line
+	3900 4500 3500 4500
+Wire Wire Line
+	3500 4600 3900 4600
+Wire Wire Line
+	3900 4700 3500 4700
+Entry Wire Line
+	4200 2900 4300 2800
+Wire Wire Line
+	4300 2800 4500 2800
+Entry Wire Line
+	4200 3000 4300 2900
+Wire Wire Line
+	4300 2900 4500 2900
+Entry Wire Line
+	4200 3100 4300 3000
+Wire Wire Line
+	4300 3000 4500 3000
+Entry Wire Line
+	4200 3200 4300 3100
+Wire Wire Line
+	4300 3100 4500 3100
+Entry Wire Line
+	4200 3300 4300 3200
+Wire Wire Line
+	4300 3200 4500 3200
+Wire Bus Line
+	4200 2550 4200 4900
+Wire Bus Line
+	4000 3100 4000 4900
+Text Label 3700 4400 0    50   ~ 0
+ROW5
+Text Label 3700 4300 0    50   ~ 0
+ROW4
+Text Label 3700 4200 0    50   ~ 0
+ROW3
+Text Label 3700 4100 0    50   ~ 0
+ROW2
+Text Label 3700 4000 0    50   ~ 0
+ROW1
+Wire Wire Line
+	3500 4400 3900 4400
+Wire Wire Line
+	3900 4300 3500 4300
+Wire Wire Line
+	3500 4200 3900 4200
+Wire Wire Line
+	3900 4100 3500 4100
+Wire Wire Line
+	3500 4000 3900 4000
+Entry Wire Line
+	3900 4400 4000 4500
+Entry Wire Line
+	3900 4300 4000 4400
+Entry Wire Line
+	3900 4200 4000 4300
+Entry Wire Line
+	3900 4100 4000 4200
+Entry Wire Line
+	3900 4000 4000 4100
 $EndSCHEMATC
