File: lh60.kicad_pcb (KiCad board)
At the start: 2 copper layers, 285 x 94.6 mm, 182 parts, among them J1 Conn_01x04, J2 Conn_01x04, P1 USB_C_Plug_USB2.0, SW1 SW_Push, U1 AMS1117-3.3, U2 STM32F103C8Tx, Y1 32.768K, Y2 8M

Commit message: 20220326 pcb init
Parts:
- removed the S77 at (176.0, 305.1)
- C5, C7: footprint Capacitor_SMD:C_0603_1608Metric_Pad1.08x0.95mm_HandSolder -> Capacitor_SMD:C_1206_3216Metric_Pad1.33x1.80mm_HandSolder
- S1, S10, S14, S15, S16, S17, S19, S20, S21, S22, S25, S26, S27, S28, S29, S30, S31, S32, S33, S34, S35, S36, S37, S38, S39, S40, S41, S42, S43, S44, S45, S46, S47, S48, S49, S5, S50, S51, S52, S53, S54, S55, S56, S57, S58, S60, S61, S62, S63, S64, S66, S67, S68, S7, S72, S74, S8, S9: footprint mx1a:KaiHua_Contact -> mx1a:KaiHua_Contact_1.00u
- S11, S13, S18, S4, S59, S6, S65, S69, S73: footprint mx1a:KaiHua_Contact -> mx1a:KaiHua_Contact_1.25u
- S12: footprint mx1a:KaiHua_Contact -> mx1a:KaiHua_Contact_2.25u
- S2, S76: footprint mx1a:KaiHua_Contact -> mx1a:KaiHua_Contact_1.50u
- S23: footprint mx1a:KaiHua_Contact -> mx1a:KaiHua_Contact_3.00u
- S24: footprint mx1a:KaiHua_Contact -> mx1a:KaiHua_Contact_6.25u
- S3, S70: footprint mx1a:KaiHua_Contact -> mx1a:KaiHua_Contact_1.75u
- S71: footprint mx1a:KaiHua_Contact -> mx1a:KaiHua_Contact_2.75u
- S75: footprint mx1a:KaiHua_Contact -> mx1a:KaiHua_Contact_2.00u
- S77: renamed from S78; footprint mx1a:KaiHua_Contact -> mx1a:KaiHua_Contact_1.25u
- S78: renamed from S79; footprint mx1a:KaiHua_Contact -> mx1a:KaiHua_Contact_ISO_Enter
- S79: renamed from S80; footprint mx1a:KaiHua_Contact -> mx1a:KaiHua_Contact_2.25u
- S80: renamed from S81; footprint mx1a:KaiHua_Contact -> mx1a:KaiHua_Contact_1.00u
- S81: renamed from S82; footprint mx1a:KaiHua_Contact -> mx1a:KaiHua_Contact_1.75u
- S82: renamed from S83; footprint mx1a:KaiHua_Contact -> mx1a:KaiHua_Contact_1.25u
- moved S60 297.9 mm to (281.9, 87.1)
- moved S78 297.8 mm to (337.1, 114.0)
- moved S49 297.1 mm to (244.2, 87.1)
- moved S79 295.0 mm to (327.2, 124.7)
- moved S62 287.3 mm to (297.8, 124.2)
- moved S29 286.0 mm to (167.8, 86.9)
- moved S74 285.3 mm to (338.6, 87.3)
- moved S35 275.5 mm to (196.6, 105.9)
- moved S3 264.3 mm to (80.3, 125.2)
- moved S50 258.6 mm to (253.9, 105.7)
- moved S57 255.5 mm to (268.0, 144.2)
- moved S71 251.7 mm to (323.2, 144.1)
- moved S51 251.4 mm to (258.4, 124.7)
- moved S11 250.2 mm to (94.5, 143.6)
- moved S48 249.3 mm to (268.3, 182.1)
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
Commit message: 20220326 pcb: keycap mount
Parts:
- removed S10, S5: MX1A, mx1a:KaiHua_Contact_1.00u
- S2: value MX1A -> locked
- S4, S69: footprint mx1a:KaiHua_Contact_1.25u -> mx1a:KaiHua_Contact_1.00u
- moved S48 34.3 mm to (239.7, 163.2)
- moved S43 25.9 mm to (220.7, 163.2)
- moved S38 25.3 mm to (201.6, 163.2), turned to 180 degrees
- moved S58 11.6 mm to (277.8, 163.2)
- moved S53 6.00 mm to (258.8, 163.2)
- moved S65 3.91 mm to (289.7, 163.2), turned to 180 degrees
- moved S64 3.06 mm to (296.9, 163.2)
- moved S69 2.57 mm to (306.4, 144.1)
- moved S4 2.53 mm to (73.0, 144.1), turned to 180 degrees
- moved S19 2.16 mm to (130.2, 87.0)
- moved S30 2.07 mm to (177.8, 106.0)
- moved S55 1.95 mm to (273.1, 106.0)
- moved S41 1.89 mm to (220.7, 125.1)
- moved S80 1.88 mm to (339.7, 144.1)
- moved S8 1.79 mm to (101.6, 106.0)
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
Commit message: 20220326 fin
Parts:
- removed J2: Conn_01x04, Connector_PinHeader_1.27mm:PinHeader_1x04_P1.27mm_Vertical
- removed S78: MX1A, mx1a:KaiHua_Contact_ISO_Enter
- added J3: Conn_01x02_Female, Connector_PinHeader_2.54mm:PinHeader_1x02_P2.54mm_Vertical, F.Cu at (129.8, 169.3)
- added J5: Conn_01x02_Female, Connector_PinHeader_2.54mm:PinHeader_1x02_P2.54mm_Vertical, F.Cu at (131.1, 165.1)
- C1, C10, C11, C12, C13, C2, C3, C4, C5, C6, C7, C8, C9, D1, D10, D11, D12, D13, D14, D15, D16, D17, D18, D19, D2, D20, D21, D22, D23, D24, D25, D26, D27, D28, D29, D3, D30, D31, D32, D33, D34, D35, D36, D37, D38, D39, D4, D40, D41, D42, D43, D44, D45, D46, D47, D48, D49, D5, D50, D51, D52, D53, D54, D55, D56, D57, D58, D59, D6, D60, D61, D62, D63, D64, D65, D66, D67, D68, D69, D7, D8, D9, P1, R1, R2, R3, R4, R5, R6, R7, R8, R9, SW1, U1, U2, Y1, Y2: moved to B.Cu
- J1: value Conn_01x04 -> Conn_01x03_Female; footprint Connector_PinHeader_1.27mm:PinHeader_1x04_P1.27mm_Vertical -> Connector_PinHeader_2.54mm:PinHeader_1x03_P2.54mm_Vertical
- S75: footprint mx1a:KaiHua_Contact_2.00u -> mx1a:KaiHua_Contact_2.00u_reverse
- moved D29 239.7 mm to (312.1, 80.7), turned to 90 degrees
- moved D69 212.9 mm to (341.2, 167.0), turned to 180 degrees
- moved D66 209.6 mm to (338.8, 109.9), turned to 180 degrees
- moved D55 196.7 mm to (286.4, 90.8), turned to 180 degrees
- moved D57 193.2 mm to (300.7, 128.9), turned to 180 degrees
- moved D62 192.5 mm to (310.5, 120.6), turned to 180 degrees
- moved D63 183.6 mm to (302.3, 148.5), turned to 180 degrees
- moved D65 178.3 mm to (334.5, 96.6), turned to -90 degrees
- moved D45 177.9 mm to (248.3, 90.8), turned to 180 degrees
- moved D50 176.0 mm to (267.3, 90.8), turned to 180 degrees
- moved D51 170.1 mm to (276.9, 109.9), turned to 180 degrees
- moved D61 169.9 mm to (315.0, 109.9), turned to 180 degrees
- moved P1 168.6 mm to (66.4, 95.6)
- moved D60 166.5 mm to (305.4, 90.8), turned to 180 degrees
- moved D54 160.4 mm to (277.1, 158.1)
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Connections:
- J1 pad 1: +3V3 -> +5V
- J1 pad 2: Net-(J1-Pad2) -> +3V3
- J1 pad 3: Net-(J1-Pad3) -> GND
- R8 pad 1: Net-(J1-Pad2) -> Net-(R8-Pad1)
- R9 pad 2: Net-(J1-Pad3) -> Net-(R9-Pad2)
- S11 pad : (no net) -> /ROW4
- S13 pad : (no net) -> /ROW5
- S18 pad : (no net) -> /ROW5
- S2 pad : (no net) -> /ROW2
- S23 pad : (no net) -> /ROW5
- S24 pad : (no net) -> /ROW5
- S3 pad : (no net) -> /ROW3
- S6 pad : (no net) -> /ROW5
- S71 pad : (no net) -> /ROW4
- S76 pad : (no net) -> /ROW2
- S77 pad : (no net) -> /ROW3
Routing:
- net /ROW5: track 0.00 -> 430.9 mm, vias 0 -> 1
- net /ROW1: track 0.00 -> 411.3 mm, vias 0 -> 2
- net /ROW2: track 0.00 -> 382.2 mm, vias 0 -> 2
- net /ROW3: track 0.00 -> 370.9 mm, vias 0 -> 3
- net /ROW4: track 0.00 -> 351.0 mm, vias 0 -> 2
- net /COL14: track 0.00 -> 309.5 mm, vias 0 -> 4
- net /COL6: track 0.00 -> 285.9 mm
- net /COL13: track 0.00 -> 245.0 mm, vias 0 -> 2
- net /COL12: track 0.00 -> 244.4 mm, vias 0 -> 2
- net /COL11: track 0.00 -> 229.4 mm, vias 0 -> 2
- net /COL9: track 0.00 -> 202.5 mm, vias 0 -> 2
- net /COL10: track 0.00 -> 197.8 mm, vias 0 -> 2
- net /COL8: track 0.00 -> 178.4 mm, vias 0 -> 2
- net /COL1: track 0.00 -> 178.1 mm, vias 0 -> 5
- net +3V3: track 0.00 -> 167.7 mm, vias 0 -> 2
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- added copper zone on B.Cu, net GND
- added copper zone on F.Cu, net GND
