File: lh60.kicad_pcb (KiCad board)
At the start: 2 copper layers, 285.8 x 95.2 mm, 0 parts

Commit message: feat(pcb): sync from sch
Parts:
- added D1: 1N4148WS, lh60-core:D_SOD-323_Bottom, F.Cu at (172.7, 83.0)
- added D10: 1N4148WS, lh60-core:D_SOD-323_Bottom, F.Cu at (172.7, 109.6)
- added D11: 1N4148WS, lh60-core:D_SOD-323_Bottom, F.Cu at (176.9, 83.0)
- added D12: 1N4148WS, lh60-core:D_SOD-323_Bottom, F.Cu at (176.9, 86.0)
- added D13: 1N4148WS, lh60-core:D_SOD-323_Bottom, F.Cu at (176.9, 88.9)
- added D14: 1N4148WS, lh60-core:D_SOD-323_Bottom, F.Cu at (176.9, 91.9)
- added D15: 1N4148WS, lh60-core:D_SOD-323_Bottom, F.Cu at (176.9, 94.8)
- added D16: 1N4148WS, lh60-core:D_SOD-323_Bottom, F.Cu at (176.9, 97.8)
- added D17: 1N4148WS, lh60-core:D_SOD-323_Bottom, F.Cu at (176.9, 100.7)
- added D18: 1N4148WS, lh60-core:D_SOD-323_Bottom, F.Cu at (176.9, 103.7)
- added D19: 1N4148WS, lh60-core:D_SOD-323_Bottom, F.Cu at (176.9, 106.6)
- added D2: 1N4148WS, lh60-core:D_SOD-323_Bottom, F.Cu at (172.7, 86.0)
- added D20: 1N4148WS, lh60-core:D_SOD-323_Bottom, F.Cu at (176.9, 109.6)
- added D21: 1N4148WS, lh60-core:D_SOD-323_Bottom, F.Cu at (181.2, 83.0)
- added D22: 1N4148WS, lh60-core:D_SOD-323_Bottom, F.Cu at (181.2, 86.0)
- added D23: 1N4148WS, lh60-core:D_SOD-323_Bottom, F.Cu at (181.2, 88.9)
- added D24: 1N4148WS, lh60-core:D_SOD-323_Bottom, F.Cu at (181.2, 91.9)
- added D25: 1N4148WS, lh60-core:D_SOD-323_Bottom, F.Cu at (181.2, 94.8)
- added D26: 1N4148WS, lh60-core:D_SOD-323_Bottom, F.Cu at (181.2, 97.8)
- added D27: 1N4148WS, lh60-core:D_SOD-323_Bottom, F.Cu at (181.2, 100.7)
- added D28: 1N4148WS, lh60-core:D_SOD-323_Bottom, F.Cu at (181.2, 103.7)
- added D29: 1N4148WS, lh60-core:D_SOD-323_Bottom, F.Cu at (181.2, 106.6)
- added D3: 1N4148WS, lh60-core:D_SOD-323_Bottom, F.Cu at (172.7, 88.9)
- added D30: 1N4148WS, lh60-core:D_SOD-323_Bottom, F.Cu at (181.2, 109.6)
- added D31: 1N4148WS, lh60-core:D_SOD-323_Bottom, F.Cu at (185.4, 83.0)
- added D32: 1N4148WS, lh60-core:D_SOD-323_Bottom, F.Cu at (185.4, 86.0)
- added D33: 1N4148WS, lh60-core:D_SOD-323_Bottom, F.Cu at (185.4, 88.9)
- added D34: 1N4148WS, lh60-core:D_SOD-323_Bottom, F.Cu at (185.4, 91.9)
- added D35: 1N4148WS, lh60-core:D_SOD-323_Bottom, F.Cu at (185.4, 94.8)
- added D36: 1N4148WS, lh60-core:D_SOD-323_Bottom, F.Cu at (185.4, 97.8)
- added D37: 1N4148WS, lh60-core:D_SOD-323_Bottom, F.Cu at (185.4, 100.7)
- added D38: 1N4148WS, lh60-core:D_SOD-323_Bottom, F.Cu at (185.4, 103.7)
- added D39: 1N4148WS, lh60-core:D_SOD-323_Bottom, F.Cu at (185.4, 106.6)
- added D4: 1N4148WS, lh60-core:D_SOD-323_Bottom, F.Cu at (172.7, 91.9)
- added D40: 1N4148WS, lh60-core:D_SOD-323_Bottom, F.Cu at (185.4, 109.6)
- added D41: 1N4148WS, lh60-core:D_SOD-323_Bottom, F.Cu at (189.7, 83.0)
- added D42: 1N4148WS, lh60-core:D_SOD-323_Bottom, F.Cu at (189.7, 86.0)
- added D43: 1N4148WS, lh60-core:D_SOD-323_Bottom, F.Cu at (189.7, 88.9)
- added D44: 1N4148WS, lh60-core:D_SOD-323_Bottom, F.Cu at (189.7, 91.9)
- added D45: 1N4148WS, lh60-core:D_SOD-323_Bottom, F.Cu at (189.7, 94.8)
- added D46: 1N4148WS, lh60-core:D_SOD-323_Bottom, F.Cu at (189.7, 97.8)
- added D47: 1N4148WS, lh60-core:D_SOD-323_Bottom, F.Cu at (189.7, 100.7)
- added D48: 1N4148WS, lh60-core:D_SOD-323_Bottom, F.Cu at (189.7, 103.7)
- added D49: 1N4148WS, lh60-core:D_SOD-323_Bottom, F.Cu at (189.7, 106.6)
- added D5: 1N4148WS, lh60-core:D_SOD-323_Bottom, F.Cu at (172.7, 94.8)
- added D50: 1N4148WS, lh60-core:D_SOD-323_Bottom, F.Cu at (189.7, 109.6)
- added D51: 1N4148WS, lh60-core:D_SOD-323_Bottom, F.Cu at (193.9, 83.0)
- added D52: 1N4148WS, lh60-core:D_SOD-323_Bottom, F.Cu at (193.9, 86.0)
- added D53: 1N4148WS, lh60-core:D_SOD-323_Bottom, F.Cu at (193.9, 88.9)
- added D54: 1N4148WS, lh60-core:D_SOD-323_Bottom, F.Cu at (193.9, 91.9)
- added D55: 1N4148WS, lh60-core:D_SOD-323_Bottom, F.Cu at (193.9, 94.8)
- added D56: 1N4148WS, lh60-core:D_SOD-323_Bottom, F.Cu at (193.9, 97.8)
- added D57: 1N4148WS, lh60-core:D_SOD-323_Bottom, F.Cu at (193.9, 100.7)
- added D58: 1N4148WS, lh60-core:D_SOD-323_Bottom, F.Cu at (193.9, 103.7)
- added D59: 1N4148WS, lh60-core:D_SOD-323_Bottom, F.Cu at (193.9, 106.6)
- added D6: 1N4148WS, lh60-core:D_SOD-323_Bottom, F.Cu at (172.7, 97.8)
- added D60: 1N4148WS, lh60-core:D_SOD-323_Bottom, F.Cu at (193.9, 109.6)
- added D61: 1N4148WS, lh60-core:D_SOD-323_Bottom, F.Cu at (198.2, 83.0)
- added D62: 1N4148WS, lh60-core:D_SOD-323_Bottom, F.Cu at (198.2, 86.0)
- added D63: 1N4148WS, lh60-core:D_SOD-323_Bottom, F.Cu at (198.2, 88.9)
- added D64: 1N4148WS, lh60-core:D_SOD-323_Bottom, F.Cu at (198.2, 91.9)
- added D65: 1N4148WS, lh60-core:D_SOD-323_Bottom, F.Cu at (198.2, 94.8)
- added D66: 1N4148WS, lh60-core:D_SOD-323_Bottom, F.Cu at (198.2, 97.8)
- added D67: 1N4148WS, lh60-core:D_SOD-323_Bottom, F.Cu at (198.2, 100.7)
- added D68: 1N4148WS, lh60-core:D_SOD-323_Bottom, F.Cu at (198.2, 103.7)
- added D69: 1N4148WS, lh60-core:D_SOD-323_Bottom, F.Cu at (198.2, 106.6)
- added D7: 1N4148WS, lh60-core:D_SOD-323_Bottom, F.Cu at (172.7, 100.7)
- added D70: 1N4148WS, lh60-core:D_SOD-323_Bottom, F.Cu at (198.2, 109.6)
- added D8: 1N4148WS, lh60-core:D_SOD-323_Bottom, F.Cu at (172.7, 103.7)
- added D9: 1N4148WS, lh60-core:D_SOD-323_Bottom, F.Cu at (172.7, 106.6)
- added SW1: r0_esc_1u, lh60-sockets:Gateron-LP-or-ChocV1-Hotswap-Socket-1U, F.Cu at (31.3, 27.8)
- added SW10: r0_9_1u, lh60-sockets:Gateron-LP-or-ChocV1-Hotswap-Socket-1U, F.Cu at (52.7, 27.8)
- added SW11: r0_0_1u, lh60-sockets:Gateron-LP-or-ChocV1-Hotswap-Socket-1U, F.Cu at (52.7, 46.0)
- added SW12: r0_minus_1u, lh60-sockets:Gateron-LP-or-ChocV1-Hotswap-Socket-1U, F.Cu at (52.7, 64.3)
- added SW13: r0_equal_1u, lh60-sockets:Gateron-LP-or-ChocV1-Hotswap-Socket-1U, F.Cu at (52.7, 82.5)
- added SW14: r0_top_2u, lh60-sockets:Gateron-LP-Hotswap-Socket-2U, F.Cu at (180.9, 22.2)
- added SW15: r0_top_split_left_fn_1u, lh60-sockets:Gateron-LP-Hotswap-Socket-1U, F.Cu at (180.9, 34.8)
- added SW16: r0_top_split_right_1u, lh60-sockets:Gateron-LP-Hotswap-Socket-1U, F.Cu at (180.9, 47.4)
- added SW17: r1_tab_1.5u, lh60-sockets:Gateron-LP-or-ChocV1-Hotswap-Socket-1.5U, F.Cu at (52.7, 100.7)
- added SW18: r1_q_1u, lh60-sockets:Gateron-LP-or-ChocV1-Hotswap-Socket-1U, F.Cu at (52.7, 119.0)
- added SW19: r1_w_1u, lh60-sockets:Gateron-LP-or-ChocV1-Hotswap-Socket-1U, F.Cu at (52.7, 137.2)
- added SW2: r0_1_1u, lh60-sockets:Gateron-LP-or-ChocV1-Hotswap-Socket-1U, F.Cu at (31.3, 46.0)
- added SW20: r1_e_1u, lh60-sockets:Gateron-LP-or-ChocV1-Hotswap-Socket-1U, F.Cu at (52.7, 155.4)
- added SW21: r1_r_1u, lh60-sockets:Gateron-LP-or-ChocV1-Hotswap-Socket-1U, F.Cu at (52.7, 173.6)
- added SW22: r1_t_1u, lh60-sockets:Gateron-LP-or-ChocV1-Hotswap-Socket-1U, F.Cu at (74.0, 27.8)
- added SW23: r1_y_1u, lh60-sockets:Gateron-LP-or-ChocV1-Hotswap-Socket-1U, F.Cu at (74.0, 46.0)
- added SW24: r1_u_1u, lh60-sockets:Gateron-LP-or-ChocV1-Hotswap-Socket-1U, F.Cu at (74.0, 64.3)
- added SW25: r1_i_1u, lh60-sockets:Gateron-LP-or-ChocV1-Hotswap-Socket-1U, F.Cu at (74.0, 82.5)
- added SW26: r1_o_1u, lh60-sockets:Gateron-LP-or-ChocV1-Hotswap-Socket-1U, F.Cu at (74.0, 100.7)
- added SW27: r1_p_1u, lh60-sockets:Gateron-LP-or-ChocV1-Hotswap-Socket-1U, F.Cu at (74.0, 119.0)
- added SW28: r1_left_bracket_1u, lh60-sockets:Gateron-LP-or-ChocV1-Hotswap-Socket-1U, F.Cu at (74.0, 137.2)
- added SW29: r1_right_bracket_1u, lh60-sockets:Gateron-LP-or-ChocV1-Hotswap-Socket-1U, F.Cu at (74.0, 155.4)
- added SW3: r0_2_1u, lh60-sockets:Gateron-LP-or-ChocV1-Hotswap-Socket-1U, F.Cu at (31.3, 64.3)
- added SW30: r1_backslash_1.5u, lh60-sockets:Gateron-LP-or-ChocV1-Hotswap-Socket-1.5U, F.Cu at (74.0, 173.6)
- added SW31: r2_caps_1.75u, lh60-sockets:Gateron-LP-or-ChocV1-Hotswap-Socket-1.75U, F.Cu at (95.4, 27.8)
- added SW32: r2_a_1u, lh60-sockets:Gateron-LP-or-ChocV1-Hotswap-Socket-1U, F.Cu at (95.4, 46.0)
- added SW33: r2_s_1u, lh60-sockets:Gateron-LP-or-ChocV1-Hotswap-Socket-1U, F.Cu at (95.4, 64.3)
- added SW34: r2_d_1u, lh60-sockets:Gateron-LP-or-ChocV1-Hotswap-Socket-1U, F.Cu at (95.4, 82.5)
- added SW35: r2_f_1u, lh60-sockets:Gateron-LP-or-ChocV1-Hotswap-Socket-1U, F.Cu at (95.4, 100.7)
- added SW36: r2_g_1u, lh60-sockets:Gateron-LP-or-ChocV1-Hotswap-Socket-1U, F.Cu at (95.4, 119.0)
- added SW37: r2_h_1u, lh60-sockets:Gateron-LP-or-ChocV1-Hotswap-Socket-1U, F.Cu at (95.4, 137.2)
- added SW38: r2_j_1u, lh60-sockets:Gateron-LP-or-ChocV1-Hotswap-Socket-1U, F.Cu at (95.4, 155.4)
- added SW39: r2_k_1u, lh60-sockets:Gateron-LP-or-ChocV1-Hotswap-Socket-1U, F.Cu at (95.4, 173.6)
- added SW4: r0_3_1u, lh60-sockets:Gateron-LP-or-ChocV1-Hotswap-Socket-1U, F.Cu at (31.3, 82.5)
- added SW40: r2_l_1u, lh60-sockets:Gateron-LP-or-ChocV1-Hotswap-Socket-1U, F.Cu at (116.8, 27.8)
- added SW41: r2_semicolon_1u, lh60-sockets:Gateron-LP-or-ChocV1-Hotswap-Socket-1U, F.Cu at (116.8, 46.0)
- added SW42: r2_quote_1u, lh60-sockets:Gateron-LP-or-ChocV1-Hotswap-Socket-1U, F.Cu at (116.8, 64.3)
- added SW43: r2_enter_ansi_2.25u, lh60-sockets:Gateron-LP-Hotswap-Socket-2.25U, F.Cu at (180.9, 60.0)
- added SW44: r2_enter_split_left_fn_1u, lh60-sockets:Gateron-LP-Hotswap-Socket-1U, F.Cu at (180.9, 72.6)
- added SW45: r2_enter_split_right_1.25u, lh60-sockets:Gateron-LP-Hotswap-Socket-1.25U, F.Cu at (199.8, 22.2)
- added SW46: r3_lshift_split_left_fn_1u, lh60-sockets:Gateron-LP-Hotswap-Socket-1U, F.Cu at (199.8, 34.8)
- added SW47: r3_lshift_2.25u, lh60-sockets:Gateron-LP-Hotswap-Socket-2.25U, F.Cu at (199.8, 47.4)
- added SW48: r3_lshift_split_1.25u, lh60-sockets:Gateron-LP-Hotswap-Socket-1.25U, F.Cu at (199.8, 60.0)
- added SW49: r3_z_1u, lh60-sockets:Gateron-LP-or-ChocV1-Hotswap-Socket-1U, F.Cu at (116.8, 82.5)
- added SW5: r0_4_1u, lh60-sockets:Gateron-LP-or-ChocV1-Hotswap-Socket-1U, F.Cu at (31.3, 100.7)
- added SW50: r3_x_1u, lh60-sockets:Gateron-LP-or-ChocV1-Hotswap-Socket-1U, F.Cu at (116.8, 100.7)
- added SW51: r3_c_1u, lh60-sockets:Gateron-LP-or-ChocV1-Hotswap-Socket-1U, F.Cu at (116.8, 119.0)
- added SW52: r3_v_1u, lh60-sockets:Gateron-LP-or-ChocV1-Hotswap-Socket-1U, F.Cu at (116.8, 137.2)
- added SW53: r3_b_1u, lh60-sockets:Gateron-LP-or-ChocV1-Hotswap-Socket-1U, F.Cu at (116.8, 155.4)
- added SW54: r3_n_1u, lh60-sockets:Gateron-LP-or-ChocV1-Hotswap-Socket-1U, F.Cu at (116.8, 173.6)
- added SW55: r3_m_1u, lh60-sockets:Gateron-LP-or-ChocV1-Hotswap-Socket-1U, F.Cu at (138.2, 27.8)
- added SW56: r3_comma_1u, lh60-sockets:Gateron-LP-or-ChocV1-Hotswap-Socket-1U, F.Cu at (138.2, 46.0)
- added SW57: r3_period_1u, lh60-sockets:Gateron-LP-or-ChocV1-Hotswap-Socket-1U, F.Cu at (138.2, 64.3)
- added SW58: r3_slash_1u, lh60-sockets:Gateron-LP-or-ChocV1-Hotswap-Socket-1U, F.Cu at (138.2, 82.5)
- added SW59: r3_rshift_2.75u, lh60-sockets:Gateron-LP-Hotswap-Socket-2.75U, F.Cu at (199.8, 72.6)
- added SW6: r0_5_1u, lh60-sockets:Gateron-LP-or-ChocV1-Hotswap-Socket-1U, F.Cu at (31.3, 119.0)
- added SW60: r3_rshift_left_1.75u, lh60-sockets:Gateron-LP-Hotswap-Socket-1.75U, F.Cu at (218.7, 22.2)
- added SW61: r3_rshift_right_fn_1u, lh60-sockets:Gateron-LP-Hotswap-Socket-1U, F.Cu at (218.7, 34.8)
- added SW62: r3_rshift_left_fn_1u, lh60-sockets:Gateron-LP-Hotswap-Socket-1U, F.Cu at (218.7, 47.4)
- added SW63: r3_rshift_right_1.75u, lh60-sockets:Gateron-LP-Hotswap-Socket-1.75U, F.Cu at (218.7, 60.0)
- added SW64: r4_left_ctrl_1.25u, lh60-sockets:Gateron-LP-or-ChocV1-Hotswap-Socket-1.25U, F.Cu at (138.2, 100.7)
- added SW65: r4_left_win_1.25u, lh60-sockets:Gateron-LP-or-ChocV1-Hotswap-Socket-1.25U, F.Cu at (138.2, 119.0)
- added SW66: r4_left_alt_1.25u, lh60-sockets:Gateron-LP-or-ChocV1-Hotswap-Socket-1.25U, F.Cu at (138.2, 137.2)
- added SW67: r4_space_2.25u, lh60-sockets:Gateron-LP-or-ChocV1-Hotswap-Socket-2.25U, F.Cu at (138.2, 155.4)
- added SW68: r4_fn_1u, lh60-sockets:Gateron-LP-or-ChocV1-Hotswap-Socket-1U, F.Cu at (138.2, 173.6)
- added SW69: r4_left_1u, lh60-sockets:Gateron-LP-or-ChocV1-Hotswap-Socket-1U, F.Cu at (159.5, 27.8)
- added SW7: r0_6_1u, lh60-sockets:Gateron-LP-or-ChocV1-Hotswap-Socket-1U, F.Cu at (31.3, 137.2)
- added SW70: r4_down_1u, lh60-sockets:Gateron-LP-or-ChocV1-Hotswap-Socket-1U, F.Cu at (159.5, 46.0)
- added SW71: r4_up_1u, lh60-sockets:Gateron-LP-or-ChocV1-Hotswap-Socket-1U, F.Cu at (159.5, 64.3)
- added SW72: r4_right_1u, lh60-sockets:Gateron-LP-or-ChocV1-Hotswap-Socket-1U, F.Cu at (159.5, 82.5)
- added SW73: r4_right_fn_1u, lh60-sockets:Gateron-LP-or-ChocV1-Hotswap-Socket-1U, F.Cu at (159.5, 100.7)
- added SW74: r4_right_alt_1u, lh60-sockets:Gateron-LP-or-ChocV1-Hotswap-Socket-1U, F.Cu at (159.5, 119.0)
- added SW75: r4_right_win_1u, lh60-sockets:Gateron-LP-or-ChocV1-Hotswap-Socket-1U, F.Cu at (159.5, 137.2)
- added SW76: r4_right_ctrl_1u, lh60-sockets:Gateron-LP-or-ChocV1-Hotswap-Socket-1U, F.Cu at (159.5, 155.4)
- added SW8: r0_7_1u, lh60-sockets:Gateron-LP-or-ChocV1-Hotswap-Socket-1U, F.Cu at (31.3, 155.4)
- added SW9: r0_8_1u, lh60-sockets:Gateron-LP-or-ChocV1-Hotswap-Socket-1U, F.Cu at (31.3, 173.6)
- added TP1: VSYS, lh60-core:TestPoint_Pad_D1.5mm_Bottom, F.Cu at (172.3, 112.8)
- added TP10: COL6, lh60-core:TestPoint_Pad_D1.5mm_Bottom, F.Cu at (176.1, 123.5)
- added TP11: COL7, lh60-core:TestPoint_Pad_D1.5mm_Bottom, F.Cu at (176.1, 127.0)
- added TP12: COL8, lh60-core:TestPoint_Pad_D1.5mm_Bottom, F.Cu at (176.1, 130.6)
- added TP13: COL9, lh60-core:TestPoint_Pad_D1.5mm_Bottom, F.Cu at (179.9, 112.8)
- added TP14: ROW0, lh60-core:TestPoint_Pad_D1.5mm_Bottom, F.Cu at (179.9, 116.4)
- added TP15: ROW1, lh60-core:TestPoint_Pad_D1.5mm_Bottom, F.Cu at (179.9, 119.9)
- added TP16: ROW2, lh60-core:TestPoint_Pad_D1.5mm_Bottom, F.Cu at (179.9, 123.5)
- added TP17: ROW3, lh60-core:TestPoint_Pad_D1.5mm_Bottom, F.Cu at (179.9, 127.0)
- added TP18: ROW4, lh60-core:TestPoint_Pad_D1.5mm_Bottom, F.Cu at (179.9, 130.6)
- added TP19: ROW5, lh60-core:TestPoint_Pad_D1.5mm_Bottom, F.Cu at (183.7, 112.8)
- added TP2: 3V3, lh60-core:TestPoint_Pad_D1.5mm_Bottom, F.Cu at (172.3, 116.4)
- added TP20: ROW6, lh60-core:TestPoint_Pad_D1.5mm_Bottom, F.Cu at (183.7, 116.4)
- added TP21: GP27, lh60-core:TestPoint_Pad_D1.5mm_Bottom, F.Cu at (183.7, 119.9)
- added TP22: GP28, lh60-core:TestPoint_Pad_D1.5mm_Bottom, F.Cu at (183.7, 123.5)
- added TP23: GP29, lh60-core:TestPoint_Pad_D1.5mm_Bottom, F.Cu at (183.7, 127.0)
- added TP3: GND, lh60-core:TestPoint_Pad_D1.5mm_Bottom, F.Cu at (172.3, 119.9)
- added TP4: COL0, lh60-core:TestPoint_Pad_D1.5mm_Bottom, F.Cu at (172.3, 123.5)
- added TP5: COL1, lh60-core:TestPoint_Pad_D1.5mm_Bottom, F.Cu at (172.3, 127.0)
- added TP6: COL2, lh60-core:TestPoint_Pad_D1.5mm_Bottom, F.Cu at (172.3, 130.6)
- added TP7: COL3, lh60-core:TestPoint_Pad_D1.5mm_Bottom, F.Cu at (176.1, 112.8)
- added TP8: COL4, lh60-core:TestPoint_Pad_D1.5mm_Bottom, F.Cu at (176.1, 116.4)
- added TP9: COL5, lh60-core:TestPoint_Pad_D1.5mm_Bottom, F.Cu at (176.1, 119.9)
- added U1: RP2040-Tiny, lh60-mcu:MCU_RP2040-Tiny_SMD, F.Cu at (210.4, 84.2)

Commit message: feat(pcb): place production sockets
Co-authored-by: TRAE CLI <noreply@bytedance.com>
Parts:
- moved SW30 245.0 mm to (271.5, 28.6)
- moved SW29 215.0 mm to (247.7, 28.6)
- moved SW9 209.8 mm to (161.9, 9.53)
- moved SW13 199.3 mm to (238.1, 9.53)
- moved SW46 192.9 mm to (9.53, 66.7), turned to 270 degrees
- moved SW28 188.9 mm to (228.6, 28.6)
- moved SW8 183.7 mm to (142.9, 9.53)
- moved SW47 179.4 mm to (21.4, 66.7)
- moved SW12 175.2 mm to (219.1, 9.53)
- moved SW48 169.0 mm to (31.0, 66.7), turned to 180 degrees
- moved SW27 162.9 mm to (209.6, 28.6)
- moved SW7 157.7 mm to (123.8, 9.53)
- moved SW11 151.8 mm to (200.0, 9.53)
- moved SW21 151.2 mm to (95.2, 28.6)
- moved SW39 149.7 mm to (176.2, 47.6)
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
Commit message: refactor(pcb): review
Parts:
- turned SW15 to 0 degrees
- turned SW43 to 180 degrees
- turned SW44 to 0 degrees
- turned SW45 to 0 degrees
- turned SW46 to 0 degrees
- turned SW47 to 180 degrees
- turned SW48 to 0 degrees

Commit message: refactor(pcb): sync & remove RShift
Parts:
- removed SW59: r3_rshift_2.75u, lh60-sockets:Gateron-LP-Hotswap-Socket-2.75U
- turned SW61 to 180 degrees
- turned SW62 to 0 degrees
- turned SW63 to 0 degrees
