File: lh60.kicad_pcb (KiCad board)
At the start: 2 copper layers, 285.8 x 95.2 mm, 169 parts, among them SW1 r0_esc_1u, SW10 r0_9_1u, SW11 r0_0_1u, SW12 r0_minus_1u, SW13 r0_equal_1u, SW14 r0_top_2u, SW15 r0_top_split_left_fn_1u, SW16 r0_top_split_right_1u, SW17 r1_tab_1.5u, SW18 r1_q_1u, SW19 r1_w_1u, SW2 r0_1_1u, SW20 r1_e_1u, SW21 r1_r_1u, SW22 r1_t_1u, SW23 r1_y_1u, SW24 r1_u_1u, SW25 r1_i_1u, SW26 r1_o_1u, SW27 r1_p_1u, SW28 r1_left_bracket_1u, SW29 r1_right_bracket_1u, SW3 r0_2_1u, SW30 r1_backslash_1.5u, SW31 r2_caps_1.75u, SW32 r2_a_1u, SW33 r2_s_1u, SW34 r2_d_1u, SW35 r2_f_1u, SW36 r2_g_1u, SW37 r2_h_1u, SW38 r2_j_1u, SW39 r2_k_1u, SW4 r0_3_1u, SW40 r2_l_1u, SW41 r2_semicolon_1u, SW42 r2_quote_1u, SW43 r2_enter_ansi_2.25u, SW44 r2_enter_split_left_fn_1u, SW45 r2_enter_split_right_1.25u, SW46 r3_lshift_split_left_fn_1u, SW47 r3_lshift_2.25u, SW48 r3_lshift_split_1.25u, SW49 r3_z_1u, SW5 r0_4_1u, SW50 r3_x_1u, SW51 r3_c_1u, SW52 r3_v_1u, SW53 r3_b_1u, SW54 r3_n_1u, SW55 r3_m_1u, SW56 r3_comma_1u, SW57 r3_period_1u, SW58 r3_slash_1u, SW6 r0_5_1u, SW60 r3_rshift_left_1.75u, SW61 r3_rshift_right_fn_1u, SW62 r3_rshift_left_fn_1u, SW63 r3_rshift_right_1.75u, SW64 r4_left_ctrl_1.25u, SW65 r4_left_win_1.25u, SW66 r4_left_alt_1.25u, SW67 r4_space_2.25u, SW68 r4_fn_1u, SW69 r4_left_1u, SW7 r0_6_1u, SW70 r4_down_1u, SW71 r4_up_1u, SW72 r4_right_1u, SW73 r4_right_fn_1u, SW74 r4_right_alt_1u, SW75 r4_right_win_1u, SW76 r4_right_ctrl_1u, SW8 r0_7_1u, SW9 r0_8_1u, U1 RP2040-Tiny

Commit message: refactor(pcb): replace test pads with debug headers
Co-authored-by: TRAE CLI <noreply@bytedance.com>
Parts:
- removed TP1: VSYS, lh60-core:TestPoint_Pad_D1.5mm_Bottom
- removed TP10: COL6, lh60-core:TestPoint_Pad_D1.5mm_Bottom
- removed TP11: COL7, lh60-core:TestPoint_Pad_D1.5mm_Bottom
- removed TP12: COL8, lh60-core:TestPoint_Pad_D1.5mm_Bottom
- removed TP13: COL9, lh60-core:TestPoint_Pad_D1.5mm_Bottom
- removed TP14: ROW0, lh60-core:TestPoint_Pad_D1.5mm_Bottom
- removed TP15: ROW1, lh60-core:TestPoint_Pad_D1.5mm_Bottom
- removed TP16: ROW2, lh60-core:TestPoint_Pad_D1.5mm_Bottom
- removed TP17: ROW3, lh60-core:TestPoint_Pad_D1.5mm_Bottom
- removed TP18: ROW4, lh60-core:TestPoint_Pad_D1.5mm_Bottom
- removed TP19: ROW5, lh60-core:TestPoint_Pad_D1.5mm_Bottom
- removed TP2: 3V3, lh60-core:TestPoint_Pad_D1.5mm_Bottom
- removed TP20: ROW6, lh60-core:TestPoint_Pad_D1.5mm_Bottom
- removed TP21: GP27, lh60-core:TestPoint_Pad_D1.5mm_Bottom
- removed TP22: GP28, lh60-core:TestPoint_Pad_D1.5mm_Bottom
- removed TP23: GP29, lh60-core:TestPoint_Pad_D1.5mm_Bottom
- removed TP3: GND, lh60-core:TestPoint_Pad_D1.5mm_Bottom
- removed TP4: COL0, lh60-core:TestPoint_Pad_D1.5mm_Bottom
- removed TP5: COL1, lh60-core:TestPoint_Pad_D1.5mm_Bottom
- removed TP6: COL2, lh60-core:TestPoint_Pad_D1.5mm_Bottom
- removed TP7: COL3, lh60-core:TestPoint_Pad_D1.5mm_Bottom
- removed TP8: COL4, lh60-core:TestPoint_Pad_D1.5mm_Bottom
- removed TP9: COL5, lh60-core:TestPoint_Pad_D1.5mm_Bottom
- added J1: PWR, lh60-core:PinHeader_1x03_P2.54mm_Vertical, F.Cu at (292.8, 5.36)
- added J2: COL_A, lh60-core:PinHeader_1x05_P2.54mm_Vertical, F.Cu at (292.8, 23.7)
- added J3: COL_B, lh60-core:PinHeader_1x05_P2.54mm_Vertical, F.Cu at (292.8, 44.5)
- added J4: ROW_A, lh60-core:PinHeader_1x04_P2.54mm_Vertical, F.Cu at (292.8, 64.1)
- added J5: ROW_B, lh60-core:PinHeader_1x03_P2.54mm_Vertical, F.Cu at (292.8, 81.2)
- added J6: AUX, lh60-core:PinHeader_1x03_P2.54mm_Vertical, F.Cu at (292.8, 97.0)

Commit message: feat(pcb): place grouped debug headers
Co-authored-by: TRAE CLI <noreply@bytedance.com>
Parts:
- J1, J2, J3, J4, J5, J6: moved to B.Cu
- moved J5 290.9 mm to (3.00, 55.5), turned to 180 degrees
- moved J4 290.1 mm to (3.00, 49.5)
- moved J2 225.8 mm to (77.5, 92.0)
- moved J3 191.2 mm to (107.5, 92.0)
- moved J6 55.9 mm to (282.5, 42.0), turned to 180 degrees
- moved J1 32.3 mm to (282.5, 36.0)
