File: lh60.kicad_sch (KiCad schematic)
At the start: 27 parts, among them J1 Conn_01x03_Female, J3 Conn_01x02_Female, J4 Conn_01x05_Socket, J5 Conn_01x02_Female, SW1 SW_Push, U1 AMS1117-3.3, U2 STM32F103C8Tx, Y1 32.768K, Y2 8M

Commit message: finish pcb v2
Parts:
- removed J3: Conn_01x02_Female, Connector_PinHeader_2.54mm:PinHeader_1x02_P2.54mm_Vertical, symbol Connector:Conn_01x02_Female
- added J2, J3: Conn_01x01_Socket, Connector_PinHeader_2.54mm:PinHeader_1x01_P2.54mm_Vertical, symbol Connector:Conn_01x01_Socket
Connections:
- net BOOT0: now also J2.1 (Pin_1)
- net BOOT1: now also J3.1 (Pin_1)
Changed lines of the file:
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@@
+    )
+  )
+  (symbol (lib_id "Connector:Conn_01x01_Socket") (at 72.39 88.9 0) (unit 1)
+    (in_bom yes) (on_board yes) (dnp no)
+    (property "Reference" "J2" (at 73.66 88.9 0)
+      (effects (font (size 1.27 1.27)) (justify left))
+    )
+    (property "Value" "Conn_01x01_Socket" (at 73.66 90.17 0)
+      (effects (font (size 1.27 1.27)) (justify left) hide)
+    )
+    (property "Footprint" "Connector_PinHeader_2.54mm:PinHeader_1x01_P2.54mm_Vertical" (at 72.39 88.9 0)
+      (effects (font (size 1.27 1.27)) hide)
+    )
+    (property "Datasheet" "~" (at 72.39 88.9 0)
+      (effects (font (size 1.27 1.27)) hide)
+    )
+    (pin "1")
+    (instances
+      (project "lh60"
+        (path "/71c31975-2c45-4d18-a25a-18e07a55d11e"
+          (reference "J2") (unit 1)
+        )
+      )
     )
   )
@@
     )
   )
-  (symbol (lib_id "Connector:Conn_01x02_Female") (at 72.39 88.9 0) (unit 1)
-    (in_bom yes) (on_board yes) (dnp no) (fields_autoplaced)
-    (property "Reference" "J3" (at 73.66 90.1699 0)
-      (effects (font (size 1.27 1.27)) (justify left))
-    )
-    (property "Value" "Conn_01x02_Female" (at 73.66 91.4399 0)
+  (symbol (lib_id "Device:R") (at 224.79 118.11 270) (unit 1)
+    (in_bom yes) (on_board yes) (dnp no)
+    (property "Reference" "R4" (at 224.79 115.57 90)
+      (effects (font (size 1.27 1.27)))
+    )
+    (property "Value" "22R" (at 224.79 118.11 90)
+      (effects (font (size 1.27 1.27)))
+    )
+    (property "Footprint" "Resistor_SMD:R_0603_1608Metric_Pad0.98x0.95mm_HandSolder" (at 224.79 116.332 90)
+      (effects (font (size 1.27 1.27)) hide)
+    )
+    (property "Datasheet" "~" (at 224.79 118.11 0)
+      (effects (font (size 1.27 1.27)) hide)
+    )
+    (pin "1")
+    (pin "2")
+    (instances
+      (project "lh60"
+        (path "/71c31975-2c45-4d18-a25a-18e07a55d11e"
+          (reference "R4") (unit 1)
+        )
+      )
+    )
+  )
+  (symbol (lib_id "Device:C") (at 54.61 134.62 90) (unit 1)
+    (in_bom yes) (on_board yes) (dnp no)
+    (property "Reference" "C2" (at 57.15 133.35 90)
+      (effects (font (size 1.27 1.27)))
+    )
+    (property "Value" "20p" (at 58.42 135.89 90)
+      (effects (font (size 1.27 1.27)))
+    )
+    (property "Footprint" "Capacitor_SMD:C_0603_1608Metric_Pad1.08x0.95mm_HandSolder" (at 58.42 133.6548 0)
+      (effects (font (size 1.27 1.27)) hide)
+    )
+    (property "Datasheet" "~" (at 54.61 134.62 0)
+      (effects (font (size 1.27 1.27)) hide)
+    )
+    (pin "1")
+    (pin "2")
+    (instances
+      (project "lh60"
+        (path "/71c31975-2c45-4d18-a25a-18e07a55d11e"
+          (reference "C2") (unit 1)
+        )
+      )
+    )
+  )
+  (symbol (lib_id "Connector:Conn_01x01_Socket") (at 72.39 91.44 0) (unit 1)
+    (in_bom yes) (on_board yes) (dnp no)
+    (property "Reference" "J3" (at 73.66 91.44 0)
+      (effects (font (size 1.27 1.27)) (justify left))
+    )
+    (property "Value" "Conn_01x01_Socket" (at 73.66 92.71 0)
       (effects (font (size 1.27 1.27)) (justify left) hide)
     )
-    (property "Footprint" "Connector_PinHeader_2.54mm:PinHeader_1x02_P2.54mm_Vertical" (at 72.39 88.9 0)
-      (effects (font (size 1.27 1.27)) hide)
-    )
-    (property "Datasheet" "~" (at 72.39 88.9 0)
-      (effects (font (size 1.27 1.27)) hide)
-    )
-    (pin "1")
-    (pin "2")
+    (property "Footprint" "Connector_PinHeader_2.54mm:PinHeader_1x01_P2.54mm_Vertical" (at 72.39 91.44 0)
+      (effects (font (size 1.27 1.27)) hide)
+    )
+    (property "Datasheet" "~" (at 72.39 91.44 0)
+      (effects (font (size 1.27 1.27)) hide)
+    )
+    (pin "1")
     (instances
       (project "lh60"
         (path "/71c31975-2c45-4d18-a25a-18e07a55d11e"
           (reference "J3") (unit 1)
-        )
-      )
-    )
-  )
-  (symbol (lib_id "Device:R") (at 224.79 118.11 270) (unit 1)
-    (in_bom yes) (on_board yes) (dnp no)
-    (property "Reference" "R4" (at 224.79 115.57 90)
-      (effects (font (size 1.27 1.27)))
-    )
-    (property "Value" "22R" (at 224.79 118.11 90)
-      (effects (font (size 1.27 1.27)))
-    )
-    (property "Footprint" "Resistor_SMD:R_0603_1608Metric_Pad0.98x0.95mm_HandSolder" (at 224.79 116.332 90)
-      (effects (font (size 1.27 1.27)) hide)
-    )
-    (property "Datasheet" "~" (at 224.79 118.11 0)
-      (effects (font (size 1.27 1.27)) hide)
-    )
-    (pin "1")
-    (pin "2")
-    (instances
-      (project "lh60"
-        (path "/71c31975-2c45-4d18-a25a-18e07a55d11e"
-          (reference "R4") (unit 1)
-        )
-      )
-    )
-  )
-  (symbol (lib_id "Device:C") (at 54.61 134.62 90) (unit 1)
-    (in_bom yes) (on_board yes) (dnp no)
-    (property "Reference" "C2" (at 57.15 133.35 90)
-      (effects (font (size 1.27 1.27)))
-    )
-    (property "Value" "20p" (at 58.42 135.89 90)
-      (effects (font (size 1.27 1.27)))
-    )
-    (property "Footprint" "Capacitor_SMD:C_0603_1608Metric_Pad1.08x0.95mm_HandSolder" (at 58.42 133.6548 0)
-      (effects (font (size 1.27 1.27)) hide)
-    )
-    (property "Datasheet" "~" (at 54.61 134.62 0)
-      (effects (font (size 1.27 1.27)) hide)
-    )
-    (pin "1")
-    (pin "2")
-    (instances
-      (project "lh60"
-        (path "/71c31975-2c45-4d18-a25a-18e07a55d11e"
-          (reference "C2") (unit 1)
         )
       )
@@
   (symbol (lib_id "Connector:Conn_01x05_Socket") (at 217.17 102.87 180) (unit 1)
     (in_bom yes) (on_board yes) (dnp no)
-    (property "Reference" "J4" (at 215.9 104.14 0)
+    (property "Reference" "J4" (at 215.9 102.87 0)
       (effects (font (size 1.27 1.27)) (justify left))
     )
     (property "Value" "Conn_01x05_Socket" (at 215.9 101.6 0)
-      (effects (font (size 1.27 1.27)) (justify left))
+      (effects (font (size 1.27 1.27)) (justify left) hide)
     )
     (property "Footprint" "USB-C:Connector-1.25-5AWT-Horizontal" (at 217.17 102.87 0)
