File: lh60.kicad_sch (KiCad schematic)
At the start: 152 parts, among them J1 PWR, J2 COL_A, J3 COL_B, J4 ROW_A, J5 ROW_B, J6 AUX, SW1 r0_esc_1u, SW10 r0_9_1u, SW11 r0_0_1u, SW12 r0_minus_1u, SW13 r0_equal_1u, SW14 r0_top_2u, SW15 r0_top_split_left_fn_1u, SW16 r0_top_split_right_1u, SW17 r1_tab_1.5u, SW18 r1_q_1u, SW19 r1_w_1u, SW2 r0_1_1u, SW20 r1_e_1u, SW21 r1_r_1u, SW22 r1_t_1u, SW23 r1_y_1u, SW24 r1_u_1u, SW25 r1_i_1u, SW26 r1_o_1u, SW27 r1_p_1u, SW28 r1_left_bracket_1u, SW29 r1_right_bracket_1u, SW3 r0_2_1u, SW30 r1_backslash_1.5u, SW31 r2_caps_1.75u, SW32 r2_a_1u, SW33 r2_s_1u, SW34 r2_d_1u, SW35 r2_f_1u, SW36 r2_g_1u, SW37 r2_h_1u, SW38 r2_j_1u, SW39 r2_k_1u, SW4 r0_3_1u, SW40 r2_l_1u, SW41 r2_semicolon_1u, SW42 r2_quote_1u, SW43 r2_enter_ansi_2.25u, SW44 r2_enter_split_left_fn_1u, SW45 r2_enter_split_right_1.25u, SW46 r3_lshift_split_left_fn_1u, SW47 r3_lshift_2.25u, SW48 r3_lshift_split_1.25u, SW49 r3_z_1u, SW5 r0_4_1u, SW50 r3_x_1u, SW51 r3_c_1u, SW52 r3_v_1u, SW53 r3_b_1u, SW54 r3_n_1u, SW55 r3_m_1u, SW56 r3_comma_1u, SW57 r3_period_1u, SW58 r3_slash_1u, SW6 r0_5_1u, SW60 r3_rshift_left_1.75u, SW61 r3_rshift_right_fn_1u, SW62 r3_rshift_left_fn_1u, SW63 r3_rshift_right_1.75u, SW64 r4_left_ctrl_1.25u, SW65 r4_left_win_1.25u, SW66 r4_left_alt_1.25u, SW67 r4_space_2.25u, SW68 r4_fn_1u, SW69 r4_left_1u, SW7 r0_6_1u, SW70 r4_down_1u, SW71 r4_up_1u, SW72 r4_right_1u, SW73 r4_right_fn_1u, SW74 r4_right_alt_1u, SW75 r4_right_win_1u, SW76 r4_right_ctrl_1u, SW8 r0_7_1u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

Commit message: feat: migrate main schematic to passive ffc
Co-authored-by: TRAE CLI <traecli@bytedance.com>
Parts:
- removed J1: PWR, lh60-core:PinHeader_1x03_P2.54mm_Vertical, symbol lh60-core:Conn_01x03
- removed J2: COL_A, lh60-core:PinHeader_1x05_P2.54mm_Vertical, symbol lh60-core:Conn_01x05
- removed J3: COL_B, lh60-core:PinHeader_1x05_P2.54mm_Vertical, symbol lh60-core:Conn_01x05
- removed J4: ROW_A, lh60-core:PinHeader_1x04_P2.54mm_Vertical, symbol lh60-core:Conn_01x04
- removed J5: ROW_B, lh60-core:PinHeader_1x03_P2.54mm_Vertical, symbol lh60-core:Conn_01x03
- removed J6: AUX, lh60-core:PinHeader_1x03_P2.54mm_Vertical, symbol lh60-core:Conn_01x03
- removed U1: RP2040-Tiny, lh60-mcu:MCU_RP2040-Tiny_SMD, symbol lh60-mcu:RP2040-Tiny
- added J1: FPC-05F-24PH20, lh60-interconnect:FPC-05F-24PH20, symbol lh60-interconnect:FPC-05F-24PH20
Connections:
- net COL0: now also J1.2
- net COL1: now also J1.3
- net COL2: now also J1.4
- net COL3: now also J1.6
- net COL4: now also J1.7
- net COL5: now also J1.8
- net COL6: now also J1.10
- net COL7: now also J1.11
- net COL8: now also J1.12
- net COL9: now also J1.13
- net GND: now also J1.1, J1.16, J1.20, J1.24, J1.5, J1.9
- net ROW0: now also J1.14
- net ROW1: now also J1.15
- net ROW2: now also J1.17
- net ROW3: now also J1.18
- net ROW4: now also J1.19
- net ROW5: now also J1.21
- net ROW6: now also J1.22
- no-connect marks 0 -> 1
